Commit message: feat(urdf): modify dynamic parameter

File: model/master_arm_pinch.urdf (robot description, URDF)
Before this commit: robot Master_Arm, 16 links, 15 joints
Links:
- link MA_Link_J1L: mass 0.23605493 -> 0.22285683
- link MA_Link_J1R: mass 0.23605493 -> 0.22285683
- link MA_Link_J2L: mass 0.25778160 -> 0.24640382
- link MA_Link_J2R: mass 0.25778160 -> 0.24640382
- link MA_Link_J3L: mass 0.22100820 -> 0.21684595
- link MA_Link_J3R: mass 0.22100820 -> 0.21684531
- link MA_Link_J4L: mass 0.16661372 -> 0.15321181
- link MA_Link_J4R: mass 0.16661372 -> 0.15321181
- link MA_Link_J5L: mass 0.22488687 -> 0.26207359
- link MA_Link_J5R: mass 0.22488687 -> 0.26207359
- link MA_Link_J6L: mass 0.16285880 -> 0.12931104
- link MA_Link_J6R: mass 0.16285880 -> 0.12931104
- link MA_Link_J7L: mass 0.19 -> 0.30239425
- link MA_Link_J7R: mass 0.19 -> 0.30239425
Joints:
- joint J10_Elbow: limit lower=-3.054326190 upper=0.087266463 effort=1000.0 velocity=3.14159265 -> lower=-0.087266463 upper=3.054326190 effort=1000.0 velocity=3.14159265; origin xyz=0.032 0.0 -0.350 rpy=0.0 0.0 0.0 -> xyz=0.032 0.0 0.230 rpy=0.0 0.0 0.0
- joint J11_Wrist_Yaw1: origin xyz=-0.032 0.0 -0.250 rpy=0.0 0.0 0.0 -> xyz=-0.032 0.0 0.245 rpy=0.0 0.0 0.0
- joint J13_Wrist_Yaw2: origin xyz=0.0 0.0 0.0 rpy=0.0 0.0 0.0 -> xyz=0.040 0.120 0.0 rpy=3.14159265 0.0 0.0
- joint J1_Shoulder_Pitch: origin xyz=0.0 -0.450 0.01 rpy=0.0 0.0 0.0 -> xyz=0.0 -0.300 0.0 rpy=0.0 0.0 0.0
- joint J4_Elbow_Pitch: origin xyz=0.032 0.0 -0.350 rpy=0.0 0.0 0.0 -> xyz=0.032 0.0 -0.230 rpy=0.0 0.0 0.0
- joint J4_Wrist_Yaw1: origin xyz=-0.032 0.0 -0.250 rpy=0.0 0.0 0.0 -> xyz=-0.032 0.0 -0.245 rpy=0.0 0.0 0.0
- joint J6_Wrist_Yaw2: origin xyz=0.0 0.0 0.0 rpy=0.0 0.0 0.0 -> xyz=0.040 0.120 0.0 rpy=0.0 0.0 0.0
- joint J7_Shoulder_Pitch: origin xyz=0.0 0.450 0.01 rpy=0.0 0.0 0.0 -> xyz=0.0 0.300 0.0 rpy=3.14159265 0.0 0.0
